File: circuit/tinyek.brd (EAGLE design)
At the start: 36.5 x 47 mm, 13 parts, among them IC1 ATTiny13A, Q1 2N7000

Commit message: update
Parts:
- C1, C2: device resistor:C050-024X044 -> c-j:50-0302-5.08
- R1: device resistor:0207/7 -> r-j:1/4W-7.62H
- R3, R4: device resistor:0204/7 -> r-j:1/4W-7.62H
Connections:
- net GND: now also C1.PAD1, C2.PAD2, R1.PAD2; no longer C1.1, C2.2, R1.2
- net N$4: now also R1.PAD1; no longer R1.1
- net N$7: now also R4.PAD2; no longer R4.2
- net N$8: now also R3.PAD2; no longer R3.2
- net N$9: now also C2.PAD1; no longer C2.1
- net VCC: now also C1.PAD2, R3.PAD1, R4.PAD1; no longer C1.2, R3.1, R4.1
Changed lines of the file:
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@@
 </element>
 <element name="G1" library="battery" package="CR2032H" value="CR2032H" x="43.18" y="40.64" rot="R270"/>
-<element name="C1" library="resistor" package="C050-024X044" value="0.1u" x="45.72" y="30.48" smashed="yes">
+<element name="C1" library="c-j" package="50-0302-5.08" value="0.1u" x="45.72" y="30.48" smashed="yes">
 <attribute name="NAME" x="43.307" y="31.623" size="1.27" layer="25" ratio="10"/>
 <attribute name="VALUE" x="43.561" y="27.813" size="1.27" layer="27" ratio="10"/>
 </element>
-<element name="C2" library="resistor" package="C050-024X044" value="0.1u" x="53.34" y="17.78" smashed="yes" rot="R270">
+<element name="C2" library="c-j" package="50-0302-5.08" value="0.1u" x="53.34" y="17.78" smashed="yes" rot="R270">
 <attribute name="NAME" x="54.737" y="18.923" size="1.27" layer="25" ratio="10" rot="R270"/>
 <attribute name="VALUE" x="50.673" y="19.939" size="1.27" layer="27" ratio="10" rot="R270"/>
 </element>
-<element name="R1" library="resistor" package="0207/7" value="470k" x="44.45" y="17.78" smashed="yes" rot="R180">
-<attribute name="NAME" x="45.72" y="18.415" size="1.27" layer="25" ratio="10" rot="R180"/>
+<element name="R1" library="r-j" package="1/4W-7.62H" value="470k" x="44.45" y="17.78" smashed="yes" rot="R180">
+<attribute name="NAME" x="39.878" y="18.415" size="1.27" layer="25" ratio="10" rot="R180"/>
 <attribute name="VALUE" x="46.736" y="18.3388" size="1.27" layer="27" ratio="10" rot="R180"/>
 </element>
@@
 </element>
 <element name="VR1" library="pot" package="B25U" value="10k" x="52.07" y="25.4" smashed="yes" rot="R270">
-<attribute name="NAME" x="52.705" y="28.448" size="1.27" layer="25" ratio="10"/>
+<attribute name="NAME" x="51.943" y="28.702" size="1.27" layer="25" ratio="10"/>
 <attribute name="VALUE" x="46.99" y="28.5496" size="1.27" layer="27" ratio="10" rot="R270"/>
 </element>
-<element name="R3" library="resistor" package="0204/7" value="2.2M" x="38.1" y="29.21" smashed="yes" rot="R270">
-<attribute name="NAME" x="37.338" y="28.9814" size="0.9906" layer="25" ratio="10"/>
+<element name="R3" library="r-j" package="1/4W-7.62H" value="2.2M" x="38.1" y="29.21" smashed="yes" rot="R270">
+<attribute name="NAME" x="37.338" y="26.6954" size="0.9906" layer="25" ratio="10"/>
 <attribute name="VALUE" x="37.6174" y="30.8356" size="0.9906" layer="27" ratio="10" rot="R270"/>
 </element>
-<element name="R4" library="resistor" package="0204/7" value="2.2M" x="35.56" y="26.67" smashed="yes" rot="R270">
-<attribute name="NAME" x="34.798" y="26.4414" size="0.9906" layer="25" ratio="10"/>
+<element name="R4" library="r-j" package="1/4W-7.62H" value="2.2M" x="35.56" y="26.67" smashed="yes" rot="R270">
+<attribute name="NAME" x="34.798" y="23.9014" size="0.9906" layer="25" ratio="10"/>
 <attribute name="VALUE" x="35.0774" y="28.2956" size="0.9906" layer="27" ratio="10" rot="R270"/>
 </element>
@@
 <signal name="GND">
 <contactref element="G1" pad="-"/>
-<contactref element="C1" pad="1"/>
+<contactref element="C1" pad="PAD1"/>
 <contactref element="IC1" pad="4"/>
 <contactref element="VR1" pad="E"/>
 <contactref element="INPUT" pad="1"/>
-<contactref element="R1" pad="2"/>
+<contactref element="R1" pad="PAD2"/>
 <contactref element="Q1" pad="1"/>
-<contactref element="C2" pad="2"/>
+<contactref element="C2" pad="PAD2"/>
 <contactref element="KEY-" pad="1"/>
 <contactref element="ISP" pad="6"/>
@@
 <contactref element="G1" pad="+"/>
 <contactref element="IC1" pad="8"/>
-<contactref element="C1" pad="2"/>
-<contactref element="R3" pad="1"/>
-<contactref element="R4" pad="1"/>
+<contactref element="C1" pad="PAD2"/>
+<contactref element="R3" pad="PAD1"/>
+<contactref element="R4" pad="PAD1"/>
 <contactref element="ISP" pad="2"/>
 <wire x1="48.26" y1="30.48" x2="58.42" y2="30.48" width="0.762" layer="16"/>
@@
 <contactref element="Q1" pad="2"/>
 <contactref element="IC1" pad="5"/>
-<contactref element="R1" pad="1"/>
+<contactref element="R1" pad="PAD1"/>
 <contactref element="ISP" pad="4"/>
 <wire x1="48.26" y1="20.32" x2="48.26" y2="17.78" width="0.762" layer="16"/>
@@
 <contactref element="IC1" pad="3"/>
 <contactref element="INPUT" pad="3"/>
-<contactref element="R4" pad="2"/>
+<contactref element="R4" pad="PAD2"/>
 <wire x1="40.64" y1="22.86" x2="35.56" y2="22.86" width="0.762" layer="16"/>
 <wire x1="35.56" y1="22.86" x2="35.56" y2="13.74" width="0.762" layer="16"/>
@@
 <contactref element="IC1" pad="2"/>
 <contactref element="INPUT" pad="2"/>
-<contactref element="R3" pad="2"/>
+<contactref element="R3" pad="PAD2"/>
 <wire x1="40.64" y1="25.4" x2="38.1" y2="25.4" width="0.762" layer="16"/>
 <wire x1="40.64" y1="25.4" x2="33.02" y2="25.4" width="0.762" layer="16"/>
@@
 <contactref element="Q1" pad="3"/>
 <contactref element="KEY+" pad="1"/>
-<contactref element="C2" pad="1"/>
+<contactref element="C2" pad="PAD1"/>
 <wire x1="53.34" y1="20.32" x2="50.8" y2="20.32" width="0.762" layer="16"/>
 <wire x1="55.88" y1="20.32" x2="53.34" y2="20.32" width="0.762" layer="16"/>
